File: Boards/VCP200 better/VCP200 better.kicad_pcb (KiCad board)
At the start: 2 copper layers, 126.2 x 71.1 mm, 65 parts, among them IC1 LM324A, IC3 VCP200, IC4 4070, IC5 4070, J1 Input Power, J2 Output, SW1 SW_MEC_5E

Commit message: fixed 4070 grounds
Connections:
- IC4 pad 7: unconnected-(IC4-Pad7) -> GND
- IC5 pad 7: unconnected-(IC5-Pad7) -> GND
