File: Boards/VCP200 better/VCP200 better.kicad_sch (KiCad schematic)
At the start: 62 parts, among them IC1 LM324A, IC3 VCP200, IC4 4070, IC5 4070, J1 Input Power, J2 Output, SW1 SW_MEC_5E

Commit message: fixed 4070 grounds
Connections:
- net GND: now also IC4.7 (VSS), IC5.7 (VSS)
Changed lines of the file:
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@@
   (junction (at 92.71 64.77) (diameter 0) (color 0 0 0 0)
   )
+  (junction (at 93.98 190.5) (diameter 0) (color 0 0 0 0)
+  )
   (junction (at 214.63 87.63) (diameter 0) (color 0 0 0 0)
   )
@@
   )
   (junction (at 80.01 190.5) (diameter 0) (color 0 0 0 0)
+  )
+  (junction (at 110.49 190.5) (diameter 0) (color 0 0 0 0)
   )
   (junction (at 116.84 62.23) (diameter 0) (color 0 0 0 0)
@@
     (stroke (width 0) (type default) (color 0 0 0 0))
   )
+  (wire (pts (xy 93.98 190.5) (xy 110.49 190.5))
+    (stroke (width 0) (type default) (color 0 0 0 0))
+  )
   (wire (pts (xy 46.99 175.26) (xy 50.8 175.26))
     (stroke (width 0) (type default) (color 0 0 0 0))
   )
-  (wire (pts (xy 86.36 190.5) (xy 119.38 190.5))
+  (wire (pts (xy 86.36 190.5) (xy 93.98 190.5))
     (stroke (width 0) (type default) (color 0 0 0 0))
   )
@@
     (stroke (width 0) (type default) (color 0 0 0 0))
   )
+  (wire (pts (xy 110.49 190.5) (xy 119.38 190.5))
+    (stroke (width 0) (type default) (color 0 0 0 0))
+  )
